Commit message: feat: refine multi-arm simulation visualization

File: pkg/src/sim/trapezoid_ur_description/urdf/trapezoid_ur7e_scene.urdf.xacro (robot description, xacro)
@@ -19,5 +19,5 @@
     sim_gazebo="$(arg sim_gazebo)"
     generate_ros2_control_tag="false">
-    <origin xyz="-0.70 -0.58 0.0" rpy="0 0 0.692"/>
+    <origin xyz="-0.70 -0.58 0.0" rpy="0 0 0"/>
   </xacro:ur_robot>
   <xacro:ur_robot
@@ -31,5 +31,5 @@
     sim_gazebo="$(arg sim_gazebo)"
     generate_ros2_control_tag="false">
-    <origin xyz="0.70 -0.58 0.0" rpy="0 0 2.450"/>
+    <origin xyz="0.70 -0.58 0.0" rpy="0 0 0"/>
   </xacro:ur_robot>
   <xacro:ur_robot
@@ -43,5 +43,5 @@
     sim_gazebo="$(arg sim_gazebo)"
     generate_ros2_control_tag="false">
-    <origin xyz="-0.32 0.58 0.0" rpy="0 0 -1.066"/>
+    <origin xyz="-0.32 0.58 0.0" rpy="0 0 0"/>
   </xacro:ur_robot>
   <xacro:ur_robot
@@ -55,5 +55,5 @@
     sim_gazebo="$(arg sim_gazebo)"
     generate_ros2_control_tag="false">
-    <origin xyz="0.32 0.58 0.0" rpy="0 0 -2.075"/>
+    <origin xyz="0.32 0.58 0.0" rpy="0 0 0"/>
   </xacro:ur_robot>
 </robot>
